Commit message: save

File: clover2_sim/clover2_description/xacro/components/motor.xacro (robot description, xacro)
@@ -1,12 +1,7 @@
-<?xml version="1.0"?>
+<?xml version="1.0" ?>
 <robot xmlns:xacro="http://ros.org/wiki/xacro">
-  <!--
-    Универсальный мотор/ротор для gz-sim (MulticopterMotorModel).
-    mesh — полный URI для атрибута mesh filename (package://.../файл).
-    Короткая форма: motor_from_package с mesh_package и mesh_file.
-  -->
   <xacro:macro
-    name="motor"
-    params="
+        name="motor"
+        params="
       parent
       motor_number
@@ -14,5 +9,4 @@
       radius_rotor
       mesh
-      mesh_scale:='1 1 1'
       name_prefix:=''
       direction:=cw
@@ -26,5 +20,4 @@
       rolling_moment_coefficient:=1e-06
       rotor_velocity_slowdown_sim:=10
-      motor_type:=velocity
       collision_length:=0.005
       visual_xyz:='0 0 0'
@@ -32,19 +25,21 @@
       inertial_xyz:='0 0 0'
       inertial_rpy:='0 0 0'
-      joint_type:=continuous
       *origin
       *inertia
     "
-  >
-    <xacro:property name="motor_link" value="${name_prefix}rotor_${motor_number}" />
-    <xacro:property name="motor_joint" value="${name_prefix}rotor_${motor_number}_joint" />
-    <joint name="${motor_joint}" type="${joint_type}">
+    >
+    <xacro:property
+            name="motor_link"
+            value="${name_prefix}rotor_${motor_number}"
+        />
+    <xacro:property
+            name="motor_joint"
+            value="${name_prefix}rotor_${motor_number}_joint"
+        />
+    <joint name="${motor_joint}" type="continuous">
       <xacro:insert_block name="origin" />
       <axis xyz="0 0 1" />
       <parent link="${parent}" />
       <child link="${motor_link}" />
-      <xacro:if value="${joint_type == 'revolute'}">
-        <limit effort="0" velocity="1000" lower="-1e+16" upper="1e+16" />
-      </xacro:if>
     </joint>
     <link name="${motor_link}">
@@ -57,16 +52,19 @@
         <origin xyz="${visual_xyz}" rpy="${visual_rpy}" />
         <geometry>
-          <mesh filename="${mesh}" scale="${mesh_scale}" />
+          <mesh filename="${mesh}" scale="1 1 1" />
         </geometry>
       </visual>
       <collision>
         <origin xyz="0 0 0" rpy="0 0 0" />
-        <geometry>
-          <cylinder length="${collision_length}" radius="${radius_rotor}" />
-        </geometry>
+          <geometry>
+            <cylinder length="${collision_length}" radius="${radius_rotor}" />
+          </geometry>
       </collision>
     </link>
     <gazebo reference="${motor_link}">
-      <plugin filename="gz-sim-multicopter-motor-model-system" name="gz::sim::systems::MulticopterMotorModel">
+      <plugin
+                filename="gz-sim-multicopter-motor-model-system"
+                name="gz::sim::systems::MulticopterMotorModel"
+            >
         <jointName>${motor_joint}</jointName>
         <linkName>${motor_link}</linkName>
@@ -80,13 +78,15 @@
         <motorNumber>${motor_number}</motorNumber>
         <rotorDragCoefficient>${rotor_drag_coefficient}</rotorDragCoefficient>
-        <rollingMomentCoefficient>${rolling_moment_coefficient}</rollingMomentCoefficient>
-        <rotorVelocitySlowdownSim>${rotor_velocity_slowdown_sim}</rotorVelocitySlowdownSim>
-        <motorType>${motor_type}</motorType>
+        <rollingMomentCoefficient
+                >${rolling_moment_coefficient}</rollingMomentCoefficient>
+        <rotorVelocitySlowdownSim
+                >${rotor_velocity_slowdown_sim}</rotorVelocitySlowdownSim>
+        <motorType>velocity</motorType>
       </plugin>
     </gazebo>
   </xacro:macro>
   <xacro:macro
-    name="motor_from_package"
-    params="
+        name="motor_from_package"
+        params="
       parent
       motor_number
@@ -95,5 +95,4 @@
       mesh_package
       mesh_file
-      mesh_scale:='1 1 1'
       name_prefix:=''
       direction:=cw
@@ -107,5 +106,4 @@
       rolling_moment_coefficient:=1e-06
       rotor_velocity_slowdown_sim:=10
-      motor_type:=velocity
       collision_length:=0.005
       visual_xyz:='0 0 0'
@@ -113,34 +111,31 @@
       inertial_xyz:='0 0 0'
       inertial_rpy:='0 0 0'
-      joint_type:=continuous
       *origin
       *inertia
     "
-  >
+    >
     <xacro:motor
-      parent="${parent}"
-      motor_number="${motor_number}"
-      mass_rotor="${mass_rotor}"
-      radius_rotor="${radius_rotor}"
-      mesh="package://${mesh_package}/${mesh_file}"
-      mesh_scale="${mesh_scale}"
-      name_prefix="${name_prefix}"
-      direction="${direction}"
-      motor_constant="${motor_constant}"
-      moment_constant="${moment_constant}"
-      time_constant_up="${time_constant_up}"
-      time_constant_down="${time_constant_down}"
-      max_rot_velocity="${max_rot_velocity}"
-      command_sub_topic="${command_sub_topic}"
-      rotor_drag_coefficient="${rotor_drag_coefficient}"
-      rolling_moment_coefficient="${rolling_moment_coefficient}"
-      rotor_velocity_slowdown_sim="${rotor_velocity_slowdown_sim}"
-      motor_type="${motor_type}"
-      collision_length="${collision_length}"
-      visual_xyz="${visual_xyz}"
-      visual_rpy="${visual_rpy}"
-      inertial_xyz="${inertial_xyz}"
-      inertial_rpy="${inertial_rpy}"
-      joint_type="${joint_type}">
+            parent="${parent}"
+            motor_number="${motor_number}"
+            mass_rotor="${mass_rotor}"
+            radius_rotor="${radius_rotor}"
+            mesh="package://${mesh_package}/${mesh_file}"
+            name_prefix="${name_prefix}"
+            direction="${direction}"
+            motor_constant="${motor_constant}"
+            moment_constant="${moment_constant}"
+            time_constant_up="${time_constant_up}"
+            time_constant_down="${time_constant_down}"
+            max_rot_velocity="${max_rot_velocity}"
+            command_sub_topic="${command_sub_topic}"
+            rotor_drag_coefficient="${rotor_drag_coefficient}"
+            rolling_moment_coefficient="${rolling_moment_coefficient}"
+            rotor_velocity_slowdown_sim="${rotor_velocity_slowdown_sim}"
+            collision_length="${collision_length}"
+            visual_xyz="${visual_xyz}"
+            visual_rpy="${visual_rpy}"
+            inertial_xyz="${inertial_xyz}"
+            inertial_rpy="${inertial_rpy}"
+        >
       <xacro:insert_block name="origin" />
       <xacro:insert_block name="inertia" />

Commit message: some xacro edit

File: clover2_sim/clover2_description/xacro/components/motor.xacro (robot description, xacro)
@@ -86,59 +86,3 @@
     </gazebo>
   </xacro:macro>
-  <xacro:macro
-        name="motor_from_package"
-        params="
-      parent
-      motor_number
-      mass_rotor
-      radius_rotor
-      mesh_package
-      mesh_file
-      name_prefix:=''
-      direction:=cw
-      motor_constant:=8.54858e-06
-      moment_constant:=0.016
-      time_constant_up:=0.0125
-      time_constant_down:=0.025
-      max_rot_velocity:=1000.0
-      command_sub_topic:=command/motor_speed
-      rotor_drag_coefficient:=8.06428e-05
-      rolling_moment_coefficient:=1e-06
-      rotor_velocity_slowdown_sim:=10
-      collision_length:=0.005
-      visual_xyz:='0 0 0'
-      visual_rpy:='0 0 0'
-      inertial_xyz:='0 0 0'
-      inertial_rpy:='0 0 0'
-      *origin
-      *inertia
-    "
-    >
-    <xacro:motor
-            parent="${parent}"
-            motor_number="${motor_number}"
-            mass_rotor="${mass_rotor}"
-            radius_rotor="${radius_rotor}"
-            mesh="package://${mesh_package}/${mesh_file}"
-            name_prefix="${name_prefix}"
-            direction="${direction}"
-            motor_constant="${motor_constant}"
-            moment_constant="${moment_constant}"
-            time_constant_up="${time_constant_up}"
-            time_constant_down="${time_constant_down}"
-            max_rot_velocity="${max_rot_velocity}"
-            command_sub_topic="${command_sub_topic}"
-            rotor_drag_coefficient="${rotor_drag_coefficient}"
-            rolling_moment_coefficient="${rolling_moment_coefficient}"
-            rotor_velocity_slowdown_sim="${rotor_velocity_slowdown_sim}"
-            collision_length="${collision_length}"
-            visual_xyz="${visual_xyz}"
-            visual_rpy="${visual_rpy}"
-            inertial_xyz="${inertial_xyz}"
-            inertial_rpy="${inertial_rpy}"
-        >
-      <xacro:insert_block name="origin" />
-      <xacro:insert_block name="inertia" />
-    </xacro:motor>
-  </xacro:macro>
 </robot>

File: clover2_sim/clover2_description/xacro/robots/clover5.urdf.xacro (robot description, xacro)
@@ -57,38 +57,30 @@
         num_motors="4"
     /> -->
-  <xacro:if value="${config['sensors']['imu']['enabled']}">
     <xacro:imu_module
-            name="imu"
+        name="imu"
+        parent="base_link"
+        mass="0.01"
+        topic="/imu/data"
+    >
+        <origin xyz="0 0 0" rpy="0 0 0" />
+    </xacro:imu_module>
+  <xacro:if value="${config['sensors']['main_camera']['enabled']}">
+    <xacro:camera_module
+            name="main_camera"
             parent="base_link"
-            xyz="${config['sensors']['imu']['position'][0]}
-             ${config['sensors']['imu']['position'][1]}
-             ${config['sensors']['imu']['position'][2]}"
-            rpy="0 0 0"
-            mass="0.01"
-            topic="/imu/data"
-        />
-  </xacro:if>
-  <xacro:if value="${config['sensors']['bottom_camera']['enabled']}">
-    <xacro:camera_module
-            name="bottom_camera"
-            parent="base_link"
-            xyz="${config['sensors']['bottom_camera']['position'][0]}
-             ${config['sensors']['bottom_camera']['position'][1]}
-             ${config['sensors']['bottom_camera']['position'][2]}"
-            rpy="${config['sensors']['bottom_camera']['orientation'][0]}
-             ${config['sensors']['bottom_camera']['orientation'][1]}
-             ${config['sensors']['bottom_camera']['orientation'][2]}"
-            width="0.03"
-            height="0.03"
-            depth="0.02"
-            mass="0.01"
             image_w="640"
             image_h="480"
             hfov="1.22"
             update_rate="30"
-            topic_rgb="/bottom_camera/image_raw"
-            topic_info="/bottom_camera/camera_info"
-            frame_optical="bottom_camera_optical_frame"
-        />
+        >
+            <origin
+                xyz="${config['sensors']['main_camera']['position'][0]}
+                     ${config['sensors']['main_camera']['position'][1]}
+                     ${config['sensors']['main_camera']['position'][2]}"
+                rpy="${config['sensors']['main_camera']['orientation'][0]}
+                     ${config['sensors']['main_camera']['orientation'][1]}
+                     ${config['sensors']['main_camera']['orientation'][2]}"
+            />
+        </xacro:camera_module>
   </xacro:if>
 </robot>

File: clover2_sim/clover2_description/xacro/robots/x500.urdf.xacro (robot description, xacro)
@@ -20,8 +20,12 @@
     />
   <xacro:include
-        filename="$(find clover2_description)/robots/xacro/x500/x500_base.xacro"
+        filename="$(find clover2_description)/xacro/robots/x500/x500_base.xacro"
     />
-  <!-- <xacro:include filename="../snippets/x500_quad_rotors.xacro" /> -->
+  <xacro:include
+        filename="$(find clover2_description)/xacro/sensors/camera_macro.xacro"
+    />
   <xacro:x500_base_link />
-  <!-- <xacro:x500_quad_rotors /> -->
+  <xacro:camera_module name="main_camera" parent="base_link">
+    <origin xyz="0 0 1" rpy="0 0 0" />
+  </xacro:camera_module>
 </robot>

File: clover2_sim/clover2_description/xacro/sensors/camera_macro.xacro (robot description, xacro)
@@ -6,13 +6,23 @@
   <xacro:macro
         name="camera_module"
-        params="name parent xyz rpy
-                       width height depth mass
-                       image_w image_h hfov update_rate
-                       topic_rgb topic_info
-                       frame_optical
-                       depth_min:=0.1 depth_max:=10.0
-                       mesh_file:=''"
+        params="
+            name
+            parent
+            name_prefix:=''
+            width:=0.01
+            height:=0.01
+            depth:=1
+            mass:=1
+            image_w:=640
+            image_h:=480
+            hfov:=2.0943951023931953
+            update_rate:=30
+            mesh_file:='file://$(find clover2_description)/meshes/sensors/camera.stl'
+            *origin
+        "
     >
-    <link name="${name}_link">
+    <xacro:property name="camera_link" value="${name_prefix}${name}" />
+    <xacro:property name="camera_joint" value="${name_prefix}${name}_joint" />
+    <link name="${camera_link}">
       <visual>
         <xacro:if value="${mesh_file == ''}">
@@ -42,17 +52,12 @@
       </xacro:box_inertial>
     </link>
-    <link name="${frame_optical}" />
-    <joint name="${name}_joint" type="fixed">
+    <joint name="${camera_joint}" type="fixed">
+      <xacro:insert_block name="origin" />
+      <axis xyz="0 0 1" />
       <parent link="${parent}" />
-      <child link="${name}_link" />
-      <origin xyz="${xyz}" rpy="${rpy}" />
+      <child link="${camera_link}" />
     </joint>
-    <joint name="${name}_optical_joint" type="fixed">
-      <parent link="${name}_link" />
-      <child link="${frame_optical}" />
-      <origin xyz="0 0 0" rpy="${-pi/2} 0 ${-pi/2}" />
-    </joint>
-    <gazebo reference="${name}_link">
-      <sensor name="${name}_rgb" type="camera">
+    <gazebo reference="${camera_link}">
+      <sensor name="${name_prefix}${name}_rgb" type="camera">
         <camera>
           <horizontal_fov>${hfov}</horizontal_fov>

File: clover2_sim/clover2_description/xacro/sensors/imu_macro.xacro (robot description, xacro)
@@ -6,15 +6,19 @@
   <xacro:macro
         name="imu_module"
-        params="name parent xyz rpy
-                       mass:=0.01
-                       size:='0.03 0.03 0.01'
-                       update_rate:=250
-                       topic:='/imu/data'
-                       frame_name:=''
-                       gyro_noise_stddev:=0.0008726646
-                       accel_xy_noise_stddev:=0.00637
-                       accel_z_noise_stddev:=0.00686
-                       visualize:=true
-                       mesh_file:=''"
+        params="
+            name
+            parent
+            mass:=0.01
+            size:='0.03 0.03 0.01'
+            update_rate:=250
+            topic:='/imu/data'
+            frame_name:=''
+            gyro_noise_stddev:=0.0008726646
+            accel_xy_noise_stddev:=0.00637
+            accel_z_noise_stddev:=0.00686
+            visualize:=true
+            mesh_file:=''
+            *origin
+        "
     >
     <xacro:property name="size_parts" value="${size.split(' ')}" />
@@ -57,5 +61,5 @@
       <parent link="${parent}" />
       <child link="${name}_link" />
-      <origin xyz="${xyz}" rpy="${rpy}" />
+      <xacro:insert_block name="origin" />
     </joint>
     <gazebo reference="${name}_link">
