Commit message: feat(description):  add physics

File: clover2_description/xacro/common/geometry.xacro (robot description, xacro)
@@ -1,7 +1,22 @@
 <?xml version="1.0"?>
 <robot xmlns:xacro="http://www.ros.org/wiki/xacro">
-  <!-- Geometry-only description: physical inertias require measured data. -->
-  <xacro:macro name="mesh_link" params="name mesh xyz:='0 0 0' rpy:='0 0 0'">
+  <!-- Approximate box inertias and collision geometry; hardware parameters are supplied by component macros. -->
+  <xacro:macro name="physical_box" params="physics">
+    <xacro:property name="m" value="${physics['mass']}"/>
+    <xacro:property name="s" value="${physics['inertia_size']}"/>
+    <inertial>
+      <origin xyz="${' '.join(str(v) for v in physics['com'])}" rpy="0 0 0"/>
+      <mass value="${m}"/>
+      <inertia ixx="${m*(s[1]**2+s[2]**2)/12}" iyy="${m*(s[0]**2+s[2]**2)/12}"
+               izz="${m*(s[0]**2+s[1]**2)/12}" ixy="0" ixz="0" iyz="0"/>
+    </inertial>
+    <collision>
+      <origin xyz="${' '.join(str(v) for v in physics['collision_xyz'])}" rpy="0 0 0"/>
+      <geometry><box size="${' '.join(str(v) for v in physics['collision_size'])}"/></geometry>
+    </collision>
+  </xacro:macro>
+  <xacro:macro name="mesh_link" params="name mesh physics xyz:='0 0 0' rpy:='0 0 0'">
     <link name="${name}">
+      <xacro:physical_box physics="${physics}"/>
       <visual>
         <origin xyz="${xyz}" rpy="${rpy}"/>

File: clover2_description/xacro/klever5/body.xacro (robot description, xacro)
@@ -2,5 +2,14 @@
 <robot xmlns:xacro="http://www.ros.org/wiki/xacro">
   <xacro:macro name="klever5_body" params="">
-    <xacro:mesh_link name="base_link" mesh="klever5/body.dae"/>
+    <!-- Body includes battery, electronics, motors and lower camera.
+         Inertia uses supplied 328x328x106 mm; collision follows mesh including legs. -->
+    <!-- Approximate hardware constants: kg, m; uniform-box inertia. -->
+    <xacro:property name="mass" value="${0.72}"/>
+    <xacro:property name="inertia_size" value="${[0.328, 0.328, 0.106]}"/>
+    <xacro:property name="com" value="${[0.0, 0.0, 0.0]}"/>
+    <xacro:property name="collision_size" value="${[0.3280731, 0.3283458, 0.2147339]}"/>
+    <xacro:property name="collision_xyz" value="${['1e-07', 0.0, '1e-07']}"/>
+    <xacro:property name="physics" value="${dict(mass=mass, inertia_size=inertia_size, com=com, collision_size=collision_size, collision_xyz=collision_xyz)}"/>
+    <xacro:mesh_link name="base_link" mesh="klever5/body.dae" physics="${physics}"/>
   </xacro:macro>
 </robot>

File: clover2_description/xacro/klever5/klever5.xacro (robot description, xacro)
@@ -14,16 +14,16 @@
   <xacro:include filename="../modules/led_strip.xacro"/>
   <xacro:klever5_body/>
-  <xacro:klever5_propellers config="${config['propellers']}"/>
+  <xacro:klever5_propellers/>
   <xacro:if value="$(arg enable_main_camera)">
-    <xacro:description_camera name="main_camera" parent="base_link" config="${config['modules']['main_camera']}"/>
+    <xacro:description_camera name="main_camera" parent="base_link" include_visual="false" include_physics="false" xyz="${config['modules']['main_camera']['xyz']}" rpy="${config['modules']['main_camera']['rpy']}"/>
   </xacro:if>
   <xacro:if value="$(arg enable_front_camera)">
-    <xacro:description_camera name="front_camera" parent="base_link" config="${config['modules']['front_camera']}"/>
+    <xacro:description_camera name="front_camera" parent="base_link" include_visual="true" include_physics="true" xyz="${config['modules']['front_camera']['xyz']}" rpy="${config['modules']['front_camera']['rpy']}"/>
   </xacro:if>
   <xacro:if value="$(arg enable_lidar)">
-    <xacro:description_lidar parent="base_link" config="${config['modules']['lidar']}"/>
+    <xacro:description_lidar parent="base_link" xyz="${config['modules']['lidar']['xyz']}" rpy="${config['modules']['lidar']['rpy']}"/>
   </xacro:if>
   <xacro:if value="$(arg enable_led_strip)">
-    <xacro:description_led_strip parent="base_link" config="${config['modules']['led_strip']}"/>
+    <xacro:description_led_strip parent="base_link" xyz="${config['modules']['led_strip']['xyz']}" rpy="${config['modules']['led_strip']['rpy']}"/>
   </xacro:if>
 </robot>

File: clover2_description/xacro/klever5/propellers.xacro (robot description, xacro)
@@ -2,12 +2,19 @@
 <robot xmlns:xacro="http://www.ros.org/wiki/xacro">
   <xacro:macro name="klever5_propeller" params="name xyz rpy">
-    <xacro:mesh_link name="${name}_link" mesh="klever5/propeller.dae"/>
+    <!-- Approximate hardware constants: kg, m; uniform-box inertia. -->
+    <xacro:property name="mass" value="${0.003}"/>
+    <xacro:property name="inertia_size" value="${[0.091603, 0.1050184, 0.008542]}"/>
+    <xacro:property name="com" value="${[-0.014212, -0.000231, 0.0]}"/>
+    <xacro:property name="collision_size" value="${[0.091603, 0.1050184, 0.008542]}"/>
+    <xacro:property name="collision_xyz" value="${[-0.014212, -0.000231, 0.0]}"/>
+    <xacro:property name="physics" value="${dict(mass=mass, inertia_size=inertia_size, com=com, collision_size=collision_size, collision_xyz=collision_xyz)}"/>
+    <xacro:mesh_link name="${name}_link" mesh="klever5/propeller.dae" physics="${physics}"/>
     <xacro:mount name="${name}_joint" parent="base_link" child="${name}_link" xyz="${xyz}" rpy="${rpy}"/>
   </xacro:macro>
-  <xacro:macro name="klever5_propellers" params="config">
-    <xacro:klever5_propeller name="propeller_front_left" xyz="${config['front_left']['xyz']}" rpy="${config['front_left']['rpy']}"/>
-    <xacro:klever5_propeller name="propeller_front_right" xyz="${config['front_right']['xyz']}" rpy="${config['front_right']['rpy']}"/>
-    <xacro:klever5_propeller name="propeller_rear_left" xyz="${config['rear_left']['xyz']}" rpy="${config['rear_left']['rpy']}"/>
-    <xacro:klever5_propeller name="propeller_rear_right" xyz="${config['rear_right']['xyz']}" rpy="${config['rear_right']['rpy']}"/>
+  <xacro:macro name="klever5_propellers" params="">
+    <xacro:klever5_propeller name="propeller_front_left" xyz="0.077 0.077 0.058" rpy="0 0 0"/>
+    <xacro:klever5_propeller name="propeller_front_right" xyz="0.077 -0.077 0.058" rpy="0 0 0"/>
+    <xacro:klever5_propeller name="propeller_rear_left" xyz="-0.077 0.077 0.058" rpy="0 0 0"/>
+    <xacro:klever5_propeller name="propeller_rear_right" xyz="-0.077 -0.077 0.058" rpy="0 0 0"/>
   </xacro:macro>
 </robot>

File: clover2_description/xacro/modules/camera.xacro (robot description, xacro)
@@ -3,10 +3,20 @@
   <!-- Body link: X forward, Y left, Z up. *_link is the optical frame
        (Z forward, X right, Y down), preserving the camera driver interface. -->
-  <xacro:macro name="description_camera" params="name parent config">
+  <xacro:macro name="description_camera" params="name parent xyz rpy include_visual:=true include_physics:=true">
+    <!-- Approximate hardware constants: kg, m; uniform-box inertia. -->
+    <xacro:property name="mass" value="${0.018}"/>
+    <xacro:property name="inertia_size" value="${[0.0174835, 0.0250188, 0.024021]}"/>
+    <xacro:property name="com" value="${['-6e-06', 0.0, 6.6e-06]}"/>
+    <xacro:property name="collision_size" value="${[0.0174835, 0.0250188, 0.024021]}"/>
+    <xacro:property name="collision_xyz" value="${['-6e-06', 0.0, 6.6e-06]}"/>
+    <xacro:property name="physics" value="${dict(mass=mass, inertia_size=inertia_size, com=com, collision_size=collision_size, collision_xyz=collision_xyz)}"/>
     <link name="${name}_body_link">
-      <xacro:if value="${config.get('mesh', '') != ''}">
+      <xacro:if value="${include_physics}">
+        <xacro:physical_box physics="${physics}"/>
+      </xacro:if>
+      <xacro:if value="${include_visual}">
         <visual>
           <geometry>
-            <mesh filename="package://clover2_description/meshes/${config['mesh']}"/>
+            <mesh filename="package://clover2_description/meshes/modules/camera.dae"/>
           </geometry>
         </visual>
@@ -14,5 +24,5 @@
     </link>
     <xacro:mount name="${name}_mount_joint" parent="${parent}" child="${name}_body_link"
-      xyz="${config['xyz']}" rpy="${config['rpy']}"/>
+      xyz="${xyz}" rpy="${rpy}"/>
     <link name="${name}_link"/>
     <xacro:mount name="${name}_optical_joint" parent="${name}_body_link" child="${name}_link"

File: clover2_description/xacro/modules/led_strip.xacro (robot description, xacro)
@@ -1,8 +1,15 @@
 <?xml version="1.0"?>
 <robot xmlns:xacro="http://www.ros.org/wiki/xacro">
-  <xacro:macro name="description_led_strip" params="parent config name:='led_strip_link'">
-    <xacro:mesh_link name="${name}" mesh="modules/led_strip.dae"/>
+  <xacro:macro name="description_led_strip" params="parent xyz rpy name:='led_strip_link'">
+    <!-- Approximate hardware constants: kg, m; uniform-box inertia. -->
+    <xacro:property name="mass" value="${0.01}"/>
+    <xacro:property name="inertia_size" value="${[0.1638838, 0.1639418, 0.0028042]}"/>
+    <xacro:property name="com" value="${[0.0, 0.0, 0.0]}"/>
+    <xacro:property name="collision_size" value="${[0.1638838, 0.1639418, 0.0028042]}"/>
+    <xacro:property name="collision_xyz" value="${[0.0, 0.0, 0.0]}"/>
+    <xacro:property name="physics" value="${dict(mass=mass, inertia_size=inertia_size, com=com, collision_size=collision_size, collision_xyz=collision_xyz)}"/>
+    <xacro:mesh_link physics="${physics}" name="${name}" mesh="modules/led_strip.dae"/>
     <xacro:mount name="${name}_joint" parent="${parent}" child="${name}"
-      xyz="${config['xyz']}" rpy="${config['rpy']}"/>
+      xyz="${xyz}" rpy="${rpy}"/>
   </xacro:macro>
 </robot>

File: clover2_description/xacro/modules/lidar.xacro (robot description, xacro)
@@ -1,8 +1,15 @@
 <?xml version="1.0"?>
 <robot xmlns:xacro="http://www.ros.org/wiki/xacro">
-  <xacro:macro name="description_lidar" params="parent config name:='laser'">
-    <xacro:mesh_link name="${name}" mesh="modules/lidar.dae"/>
+  <xacro:macro name="description_lidar" params="parent xyz rpy name:='laser'">
+    <!-- Approximate hardware constants: kg, m; uniform-box inertia. -->
+    <xacro:property name="mass" value="${0.1}"/>
+    <xacro:property name="inertia_size" value="${[0.0837121, 0.0556375, 0.1242414]}"/>
+    <xacro:property name="com" value="${[-0.0149865, 1.12e-05, -0.0500253]}"/>
+    <xacro:property name="collision_size" value="${[0.0837121, 0.0556375, 0.1242414]}"/>
+    <xacro:property name="collision_xyz" value="${[-0.0149865, 1.12e-05, -0.0500253]}"/>
+    <xacro:property name="physics" value="${dict(mass=mass, inertia_size=inertia_size, com=com, collision_size=collision_size, collision_xyz=collision_xyz)}"/>
+    <xacro:mesh_link physics="${physics}" name="${name}" mesh="modules/lidar.dae"/>
     <xacro:mount name="${name}_joint" parent="${parent}" child="${name}"
-      xyz="${config['xyz']}" rpy="${config['rpy']}"/>
+      xyz="${xyz}" rpy="${rpy}"/>
   </xacro:macro>
 </robot>

Commit message: feat(sim): add configurable Klever5 Gazebo description

File: clover2_description/xacro/common/geometry.xacro (robot description, xacro)
@@ -1,14 +1,8 @@
 <?xml version="1.0"?>
 <robot xmlns:xacro="http://www.ros.org/wiki/xacro">
+  <xacro:include filename="common.xacro"/>
   <!-- Approximate box inertias and collision geometry; hardware parameters are supplied by component macros. -->
   <xacro:macro name="physical_box" params="physics">
-    <xacro:property name="m" value="${physics['mass']}"/>
-    <xacro:property name="s" value="${physics['inertia_size']}"/>
-    <inertial>
-      <origin xyz="${' '.join(str(v) for v in physics['com'])}" rpy="0 0 0"/>
-      <mass value="${m}"/>
-      <inertia ixx="${m*(s[1]**2+s[2]**2)/12}" iyy="${m*(s[0]**2+s[2]**2)/12}"
-               izz="${m*(s[0]**2+s[1]**2)/12}" ixy="0" ixz="0" iyz="0"/>
-    </inertial>
+    <xacro:box_inertial physics="${physics}" format="urdf"/>
     <collision>
       <origin xyz="${' '.join(str(v) for v in physics['collision_xyz'])}" rpy="0 0 0"/>

File: clover2_description/xacro/klever5/body.xacro (robot description, xacro)
@@ -1,15 +1,8 @@
 <?xml version="1.0"?>
 <robot xmlns:xacro="http://www.ros.org/wiki/xacro">
-  <xacro:macro name="klever5_body" params="">
-    <!-- Body includes battery, electronics, motors and lower camera.
-         Inertia uses supplied 328x328x106 mm; collision follows mesh including legs. -->
-    <!-- Approximate hardware constants: kg, m; uniform-box inertia. -->
-    <xacro:property name="mass" value="${0.72}"/>
-    <xacro:property name="inertia_size" value="${[0.328, 0.328, 0.106]}"/>
-    <xacro:property name="com" value="${[0.0, 0.0, 0.0]}"/>
-    <xacro:property name="collision_size" value="${[0.3280731, 0.3283458, 0.2147339]}"/>
-    <xacro:property name="collision_xyz" value="${['1e-07', 0.0, '1e-07']}"/>
-    <xacro:property name="physics" value="${dict(mass=mass, inertia_size=inertia_size, com=com, collision_size=collision_size, collision_xyz=collision_xyz)}"/>
-    <xacro:mesh_link name="base_link" mesh="klever5/body.dae" physics="${physics}"/>
+  <xacro:include filename="../common/geometry.xacro"/>
+  <xacro:macro name="klever5_body" params="body name:=base_link">
+    <xacro:property name="physics" value="${dict(mass=body['mass'], inertia_size=body['inertia_size'], com=body['com'], collision_size=body['collision_size'], collision_xyz=body['collision_xyz'])}"/>
+    <xacro:mesh_link name="${name}" mesh="${body['mesh']}" physics="${physics}"/>
   </xacro:macro>
 </robot>

File: clover2_description/xacro/klever5/klever5.xacro (robot description, xacro)
@@ -13,6 +13,6 @@
   <xacro:include filename="../modules/lidar.xacro"/>
   <xacro:include filename="../modules/led_strip.xacro"/>
-  <xacro:klever5_body/>
-  <xacro:klever5_propellers/>
+  <xacro:klever5_body body="${config['body']}"/>
+  <xacro:klever5_propellers propeller="${config['propeller']}" rotors="${config['rotors']}"/>
   <xacro:if value="$(arg enable_main_camera)">
     <xacro:description_camera name="main_camera" parent="base_link" include_visual="false" include_physics="false" xyz="${config['modules']['main_camera']['xyz']}" rpy="${config['modules']['main_camera']['rpy']}"/>

File: clover2_description/xacro/klever5/propellers.xacro (robot description, xacro)
@@ -1,20 +1,15 @@
 <?xml version="1.0"?>
 <robot xmlns:xacro="http://www.ros.org/wiki/xacro">
-  <xacro:macro name="klever5_propeller" params="name xyz rpy">
-    <!-- Approximate hardware constants: kg, m; uniform-box inertia. -->
-    <xacro:property name="mass" value="${0.003}"/>
-    <xacro:property name="inertia_size" value="${[0.091603, 0.1050184, 0.008542]}"/>
-    <xacro:property name="com" value="${[-0.014212, -0.000231, 0.0]}"/>
-    <xacro:property name="collision_size" value="${[0.091603, 0.1050184, 0.008542]}"/>
-    <xacro:property name="collision_xyz" value="${[-0.014212, -0.000231, 0.0]}"/>
-    <xacro:property name="physics" value="${dict(mass=mass, inertia_size=inertia_size, com=com, collision_size=collision_size, collision_xyz=collision_xyz)}"/>
-    <xacro:mesh_link name="${name}_link" mesh="klever5/propeller.dae" physics="${physics}"/>
-    <xacro:mount name="${name}_joint" parent="base_link" child="${name}_link" xyz="${xyz}" rpy="${rpy}"/>
+  <xacro:include filename="../common/geometry.xacro"/>
+  <xacro:macro name="klever5_propeller" params="name parent propeller xyz rpy">
+    <xacro:property name="physics" value="${dict(mass=propeller['mass'], inertia_size=propeller['inertia_size'], com=propeller['com'], collision_size=propeller['collision_size'], collision_xyz=propeller['collision_xyz'])}"/>
+    <xacro:mesh_link name="${name}_link" mesh="${propeller['mesh']}" physics="${physics}"/>
+    <xacro:mount name="${name}_joint" parent="${parent}" child="${name}_link" xyz="${xyz}" rpy="${rpy}"/>
   </xacro:macro>
-  <xacro:macro name="klever5_propellers" params="">
-    <xacro:klever5_propeller name="propeller_front_left" xyz="0.077 0.077 0.058" rpy="0 0 0"/>
-    <xacro:klever5_propeller name="propeller_front_right" xyz="0.077 -0.077 0.058" rpy="0 0 0"/>
-    <xacro:klever5_propeller name="propeller_rear_left" xyz="-0.077 0.077 0.058" rpy="0 0 0"/>
-    <xacro:klever5_propeller name="propeller_rear_right" xyz="-0.077 -0.077 0.058" rpy="0 0 0"/>
+  <xacro:macro name="klever5_propellers" params="propeller rotors parent:=base_link prefix:=''">
+    <xacro:klever5_propeller propeller="${propeller}" parent="${parent}" name="${prefix}propeller_front_left" xyz="${rotors['front_left']['xyz']}" rpy="${rotors['front_left']['rpy']}"/>
+    <xacro:klever5_propeller propeller="${propeller}" parent="${parent}" name="${prefix}propeller_front_right" xyz="${rotors['front_right']['xyz']}" rpy="${rotors['front_right']['rpy']}"/>
+    <xacro:klever5_propeller propeller="${propeller}" parent="${parent}" name="${prefix}propeller_rear_left" xyz="${rotors['rear_left']['xyz']}" rpy="${rotors['rear_left']['rpy']}"/>
+    <xacro:klever5_propeller propeller="${propeller}" parent="${parent}" name="${prefix}propeller_rear_right" xyz="${rotors['rear_right']['xyz']}" rpy="${rotors['rear_right']['rpy']}"/>
   </xacro:macro>
 </robot>

File: clover2_description/xacro/modules/camera.xacro (robot description, xacro)
@@ -1,14 +1,9 @@
 <?xml version="1.0"?>
 <robot xmlns:xacro="http://www.ros.org/wiki/xacro">
+  <xacro:include filename="../common/geometry.xacro"/>
   <!-- Body link: X forward, Y left, Z up. *_link is the optical frame
        (Z forward, X right, Y down), preserving the camera driver interface. -->
   <xacro:macro name="description_camera" params="name parent xyz rpy include_visual:=true include_physics:=true">
-    <!-- Approximate hardware constants: kg, m; uniform-box inertia. -->
-    <xacro:property name="mass" value="${0.018}"/>
-    <xacro:property name="inertia_size" value="${[0.0174835, 0.0250188, 0.024021]}"/>
-    <xacro:property name="com" value="${['-6e-06', 0.0, 6.6e-06]}"/>
-    <xacro:property name="collision_size" value="${[0.0174835, 0.0250188, 0.024021]}"/>
-    <xacro:property name="collision_xyz" value="${['-6e-06', 0.0, 6.6e-06]}"/>
-    <xacro:property name="physics" value="${dict(mass=mass, inertia_size=inertia_size, com=com, collision_size=collision_size, collision_xyz=collision_xyz)}"/>
+    <xacro:property name="physics" value="${component_physics['camera']}"/>
     <link name="${name}_body_link">
       <xacro:if value="${include_physics}">

File: clover2_description/xacro/modules/led_strip.xacro (robot description, xacro)
@@ -1,12 +1,7 @@
 <?xml version="1.0"?>
 <robot xmlns:xacro="http://www.ros.org/wiki/xacro">
+  <xacro:include filename="../common/geometry.xacro"/>
   <xacro:macro name="description_led_strip" params="parent xyz rpy name:='led_strip_link'">
-    <!-- Approximate hardware constants: kg, m; uniform-box inertia. -->
-    <xacro:property name="mass" value="${0.01}"/>
-    <xacro:property name="inertia_size" value="${[0.1638838, 0.1639418, 0.0028042]}"/>
-    <xacro:property name="com" value="${[0.0, 0.0, 0.0]}"/>
-    <xacro:property name="collision_size" value="${[0.1638838, 0.1639418, 0.0028042]}"/>
-    <xacro:property name="collision_xyz" value="${[0.0, 0.0, 0.0]}"/>
-    <xacro:property name="physics" value="${dict(mass=mass, inertia_size=inertia_size, com=com, collision_size=collision_size, collision_xyz=collision_xyz)}"/>
+    <xacro:property name="physics" value="${component_physics['led_strip']}"/>
     <xacro:mesh_link physics="${physics}" name="${name}" mesh="modules/led_strip.dae"/>
     <xacro:mount name="${name}_joint" parent="${parent}" child="${name}"

File: clover2_description/xacro/modules/lidar.xacro (robot description, xacro)
@@ -1,12 +1,7 @@
 <?xml version="1.0"?>
 <robot xmlns:xacro="http://www.ros.org/wiki/xacro">
+  <xacro:include filename="../common/geometry.xacro"/>
   <xacro:macro name="description_lidar" params="parent xyz rpy name:='laser'">
-    <!-- Approximate hardware constants: kg, m; uniform-box inertia. -->
-    <xacro:property name="mass" value="${0.1}"/>
-    <xacro:property name="inertia_size" value="${[0.0837121, 0.0556375, 0.1242414]}"/>
-    <xacro:property name="com" value="${[-0.0149865, 1.12e-05, -0.0500253]}"/>
-    <xacro:property name="collision_size" value="${[0.0837121, 0.0556375, 0.1242414]}"/>
-    <xacro:property name="collision_xyz" value="${[-0.0149865, 1.12e-05, -0.0500253]}"/>
-    <xacro:property name="physics" value="${dict(mass=mass, inertia_size=inertia_size, com=com, collision_size=collision_size, collision_xyz=collision_xyz)}"/>
+    <xacro:property name="physics" value="${component_physics['lidar']}"/>
     <xacro:mesh_link physics="${physics}" name="${name}" mesh="modules/lidar.dae"/>
     <xacro:mount name="${name}_joint" parent="${parent}" child="${name}"
