Commit message: feat(description): update Klever5 meshes and body pose

File: clover2_description/gazebo/klever5/klever5.sdf.xacro (robot description, xacro)
@@ -23,4 +23,5 @@
       <gravity>true</gravity>
       <visual name="body_visual">
+        <pose>${body['xyz']} ${body['rpy']}</pose>
         <geometry>
           <mesh><uri>file://${description_share}/meshes/${body['mesh']}</uri></mesh>

File: clover2_description/xacro/klever5/body.xacro (robot description, xacro)
@@ -2,7 +2,7 @@
 <robot xmlns:xacro="http://www.ros.org/wiki/xacro">
   <xacro:include filename="../common/geometry.xacro"/>
-  <xacro:macro name="klever5_body" params="body name:=base_link">
+  <xacro:macro name="klever5_body" params="body xyz:='0 0 0' rpy:='0 0 0' name:=base_link">
     <xacro:property name="physics" value="${dict(mass=body['mass'], inertia_size=body['inertia_size'], com=body['com'], collision_size=body['collision_size'], collision_xyz=body['collision_xyz'])}"/>
-    <xacro:mesh_link name="${name}" mesh="${body['mesh']}" physics="${physics}"/>
+    <xacro:mesh_link name="${name}" mesh="${body['mesh']}" physics="${physics}" xyz="${xyz}" rpy="${rpy}"/>
   </xacro:macro>
 </robot>

File: clover2_description/xacro/klever5/klever5.xacro (robot description, xacro)
@@ -13,5 +13,5 @@
   <xacro:include filename="../modules/lidar.xacro"/>
   <xacro:include filename="../modules/led_strip.xacro"/>
-  <xacro:klever5_body body="${config['body']}"/>
+  <xacro:klever5_body body="${config['body']}" xyz="${config['body']['xyz']}" rpy="${config['body']['rpy']}"/>
   <xacro:klever5_propellers propeller="${config['propeller']}" rotors="${config['rotors']}"/>
   <xacro:if value="$(arg enable_main_camera)">

Commit message: feat(sim): add procedural LED strip visuals and plugin

File: clover2_description/gazebo/klever5/klever5.sdf.xacro (robot description, xacro)
@@ -16,4 +16,5 @@
   <xacro:include filename="sensors.xacro"/>
   <xacro:include filename="modules.xacro"/>
+  <xacro:include filename="led_strip.xacro"/>
   <model name="klever5">
     <static>false</static>
@@ -59,8 +60,6 @@
     </xacro:if>
     <xacro:if value="$(arg enable_led_strip)">
-      <xacro:sdf_component name="led_strip_link" parent="base_link" mount="${config['modules']['led_strip']}"
-        physics="${component_physics['led_strip']}" description_share="${description_share}">
-        <gravity>true</gravity>
-      </xacro:sdf_component>
+      <xacro:sdf_led_strip parent="base_link" mount="${config['modules']['led_strip']}"
+        physics="${component_physics['led_strip']}"/>
     </xacro:if>
   </model>

File: clover2_description/xacro/modules/led_strip.xacro (robot description, xacro)
@@ -4,5 +4,7 @@
   <xacro:macro name="description_led_strip" params="parent xyz rpy name:='led_strip_link'">
     <xacro:property name="physics" value="${component_physics['led_strip']}"/>
-    <xacro:mesh_link physics="${physics}" name="${name}" mesh="modules/led_strip.glb"/>
+    <link name="${name}">
+      <xacro:physical_box physics="${physics}"/>
+    </link>
     <xacro:mount name="${name}_joint" parent="${parent}" child="${name}"
       xyz="${xyz}" rpy="${rpy}"/>

Commit message: feat: cpu rangefinder and split xacro

File: clover2_description/gazebo/klever5/klever5.sdf.xacro (robot description, xacro)
@@ -8,4 +8,7 @@
   <xacro:arg name="enable_lidar" default="false"/>
   <xacro:arg name="enable_led_strip" default="false"/>
+  <xacro:arg name="rangefinder_type" default="raycast"/>
+  <!-- index validates the choice, including when xacro is invoked directly. -->
+  <xacro:property name="use_gpu_rangefinder" value="${['raycast', 'gpu_lidar'].index('$(arg rangefinder_type)') == 1}"/>
   <xacro:property name="description_share" value="$(arg description_share)"/>
   <xacro:property name="config" value="${xacro.load_yaml('$(arg config_file)')}"/>
@@ -14,5 +17,5 @@
   <xacro:include filename="../../xacro/common/common.xacro"/>
   <xacro:include filename="rotors.xacro"/>
-  <xacro:include filename="sensors.xacro"/>
+  <xacro:include filename="sensors/*.xacro"/>
   <xacro:include filename="modules.xacro"/>
   <xacro:include filename="led_strip.xacro"/>
@@ -33,5 +36,8 @@
         <geometry><box><size>${' '.join(str(value) for value in body['collision_size'])}</size></box></geometry>
       </collision>
-      <xacro:klever5_gazebo_sensors/>
+      <xacro:sdf_px4_sensors/>
+      <xacro:if value="${use_gpu_rangefinder}">
+        <xacro:sdf_gpu_rangefinder_sensor/>
+      </xacro:if>
       <xacro:if value="$(arg enable_main_camera)">
         <xacro:sdf_camera_sensor name="main_camera" settings="${config['simulation']['camera']}"
@@ -39,4 +45,7 @@
       </xacro:if>
     </link>
+    <xacro:unless value="${use_gpu_rangefinder}">
+      <xacro:sdf_raycast_rangefinder_plugin/>
+    </xacro:unless>
     <xacro:klever5_gazebo_rotors config="${config}" description_share="${description_share}"/>
     <xacro:if value="$(arg enable_main_camera)">

File: clover2_description/gazebo/klever5/sensors/px4.xacro (robot description, xacro)
@@ -2,5 +2,5 @@
 <sdf xmlns:xacro="http://www.ros.org/wiki/xacro" version="1.9">
   <!-- Sensor names are part of the PX4 Gazebo bridge interface. -->
-  <xacro:macro name="klever5_gazebo_sensors" params="">
+  <xacro:macro name="sdf_px4_sensors" params="">
     <sensor name="air_pressure_sensor" type="air_pressure">
       <always_on>1</always_on><update_rate>50</update_rate>
@@ -33,30 +33,4 @@
       <always_on>1</always_on><update_rate>30</update_rate>
     </sensor>
-    <sensor name="rangefinder" type="gpu_lidar">
-      <pose>0.025 0 -0.03 0 1.5707 3.1415926</pose>
-      <always_on>true</always_on>
-      <update_rate>10</update_rate>
-      <visualize>false</visualize>
-      <ray>
-        <scan>
-          <horizontal>
-            <samples>10</samples>
-            <resolution>1</resolution>
-            <min_angle>-0.0872</min_angle>
-            <max_angle>0.0872</max_angle>
-          </horizontal>
-        </scan>
-        <range>
-          <min>0.1</min>
-          <max>30</max>
-          <resolution>0.01</resolution>
-        </range>
-        <noise>
-          <type>gaussian</type>
-          <mean>0.0</mean>
-          <stddev>0.01</stddev>
-        </noise>
-      </ray>
-    </sensor>
   </xacro:macro>
 </sdf>

Commit message: move under custom sensor

File: clover2_description/gazebo/klever5/klever5.sdf.xacro (robot description, xacro)
@@ -40,4 +40,7 @@
         <xacro:sdf_gpu_rangefinder_sensor/>
       </xacro:if>
+      <xacro:unless value="${use_gpu_rangefinder}">
+        <xacro:sdf_raycast_rangefinder_sensor/>
+      </xacro:unless>
       <xacro:if value="$(arg enable_main_camera)">
         <xacro:sdf_camera_sensor name="main_camera" settings="${config['simulation']['camera']}"
@@ -45,7 +48,4 @@
       </xacro:if>
     </link>
-    <xacro:unless value="${use_gpu_rangefinder}">
-      <xacro:sdf_raycast_rangefinder_plugin/>
-    </xacro:unless>
     <xacro:klever5_gazebo_rotors config="${config}" description_share="${description_share}"/>
     <xacro:if value="$(arg enable_main_camera)">

File: clover2_description/gazebo/klever5/sensors/rangefinder.xacro (robot description, xacro)
@@ -29,18 +29,20 @@
     </sensor>
   </xacro:macro>
-  <xacro:macro name="sdf_raycast_rangefinder_plugin" params="">
-    <!-- Physics rangefinder from clover2-sim; works with Ogre1 and Ogre2. -->
-    <plugin filename="clover2-rangefinder-system" name="clover2::sim::RangefinderSystem">
-      <link_name>base_link</link_name>
-      <frame_name>main_camera_link</frame_name>
+  <xacro:macro name="sdf_raycast_rangefinder_sensor" params="">
+    <!-- Gazebo loads the system plugin from this custom sensor under a link. -->
+    <sensor name="rangefinder" type="custom">
       <pose>0.025 0 -0.03 0 1.5707 3.1415926</pose>
-      <samples>10</samples>
-      <min_angle>-0.0872</min_angle>
-      <max_angle>0.0872</max_angle>
-      <min_range>0.1</min_range>
-      <max_range>30</max_range>
+      <always_on>true</always_on>
       <update_rate>10</update_rate>
-      <noise_stddev>0.01</noise_stddev>
-    </plugin>
+      <plugin filename="clover2_gz_sim_rangefinder_system" name="clover2::sim::RangefinderSystem">
+        <frame_name>main_camera_link</frame_name>
+        <samples>10</samples>
+        <min_angle>-0.0872</min_angle>
+        <max_angle>0.0872</max_angle>
+        <min_range>0.1</min_range>
+        <max_range>30</max_range>
+        <noise_stddev>0.01</noise_stddev>
+      </plugin>
+    </sensor>
   </xacro:macro>
 </sdf>

Commit message: feat: add raycast rangefinder for OGRE1 (#69)
* feat: cpu rangefinder and split xacro

* move under custom sensor

File: clover2_description/gazebo/klever5/klever5.sdf.xacro (robot description, xacro)
@@ -8,4 +8,7 @@
   <xacro:arg name="enable_lidar" default="false"/>
   <xacro:arg name="enable_led_strip" default="false"/>
+  <xacro:arg name="rangefinder_type" default="raycast"/>
+  <!-- index validates the choice, including when xacro is invoked directly. -->
+  <xacro:property name="use_gpu_rangefinder" value="${['raycast', 'gpu_lidar'].index('$(arg rangefinder_type)') == 1}"/>
   <xacro:property name="description_share" value="$(arg description_share)"/>
   <xacro:property name="config" value="${xacro.load_yaml('$(arg config_file)')}"/>
@@ -14,5 +17,5 @@
   <xacro:include filename="../../xacro/common/common.xacro"/>
   <xacro:include filename="rotors.xacro"/>
-  <xacro:include filename="sensors.xacro"/>
+  <xacro:include filename="sensors/*.xacro"/>
   <xacro:include filename="modules.xacro"/>
   <xacro:include filename="led_strip.xacro"/>
@@ -33,5 +36,11 @@
         <geometry><box><size>${' '.join(str(value) for value in body['collision_size'])}</size></box></geometry>
       </collision>
-      <xacro:klever5_gazebo_sensors/>
+      <xacro:sdf_px4_sensors/>
+      <xacro:if value="${use_gpu_rangefinder}">
+        <xacro:sdf_gpu_rangefinder_sensor/>
+      </xacro:if>
+      <xacro:unless value="${use_gpu_rangefinder}">
+        <xacro:sdf_raycast_rangefinder_sensor/>
+      </xacro:unless>
       <xacro:if value="$(arg enable_main_camera)">
         <xacro:sdf_camera_sensor name="main_camera" settings="${config['simulation']['camera']}"
